File: Logo/Forgotten Machines Logo.kicad_pcb (KiCad board)
At the start: 2 copper layers, 0 parts

Commit message: experiments
Other:
- board text added: "0.05 Import Scale 0.5 Default Line Width"
- board text added: "0.1 Import Scale"
- board text added: "0.125 Import Scale"
- board text added: "0.125 Import Scale 0.5 Default Line Width"
- board text added: "0.125 Import Scale 5 Default Line Width"
- board text added: "2.4 Import Scale 0.05 Default Line Width"
- board text added: "Forgotten Machines Logo - Center Color Removed Trace Bitmap.dxf"
- board text added: "Forgotten Machines Logo - Hand Traced.dxf"
- board text added: "Forgotten Machines Logo - Inner-Single-Line Trace Bitmap.dxf"
- board text added: "Forgotten Machines Logo - Inner-Single-Line Trace Bitmap.svg"
- board text added: "Forgotten Machines Logo - Outer-Single-Line Trace Bitmap.dxf"
