File: Logo/Forgotten Machines Logo.kicad_pcb (KiCad board)
At the start: 2 copper layers, 0 parts

Commit message: o
Other:
- board text added: "0.01 Import Scale"
- board text added: "0.025 Import Scale"
- board text added: "0.05 Import Scale"
