File: DIP Socket Adaptor - EEPROM/2716 to 82S129.kicad_sch (KiCad schematic)
At the start: 0 parts

Commit message: 82S129/6
Parts:
- added U1: 2716_EPROM, Package_DIP:DIP-24_W15.24mm, symbol ForgottenMachines:2716_EPROM
- added U2: 82S126, Package_DIP:DIP-16_W7.62mm, symbol ForgottenMachines:82S126
Connections:
- new net +24V: U1.21 (Vpp)
- new net +5V: U1.24 (VCC), U2.16 (VCC)
- new net A0: U1.8 (A0), U2.5 (A0)
- new net A1: U1.7 (A1), U2.6 (A1)
- new net A2: U1.6 (A2), U2.7 (A2)
- new net A3: U1.5 (A3), U2.4 (A3)
- new net A4: U1.4 (A4), U2.3 (A4)
- new net A5: U1.3 (A5), U2.2 (A5)
- new net A6: U1.2 (A6), U2.1 (A6)
- new net A7: U1.1 (A7), U2.15 (A7)
- new net GND: U1.12 (GND), U1.14 (O4), U1.15 (O5), U1.16 (O6), U1.17 (O7), U2.8 (GND)
- new net O1: U1.9 (O0), U2.12 (O1)
- new net O2: U1.10 (O1), U2.11 (O2)
- new net O3: U1.11 (O2), U2.10 (O3)
- new net O4: U1.13 (O3), U2.9 (O4)
- new net ~{CE1}: U1.20 (~{OE}), U2.13 (~{CE1}), U2.14 (~{CE2})
- no-connect marks 0 -> 4
