File: DIP Socket Adaptor - EEPROM/EPROM 2716 Program Voltage Booster.kicad_sch (KiCad schematic)
At the start: 8 parts, among them J1 External Power for Vpp, P1 2716_EPROM, SW1 Voltage Boost, U1 2716_EPROM

Commit message: 2716 Vpp boost
Parts:
- J1: footprint (none) -> Connector_PinHeader_2.54mm:PinHeader_1x04_P2.54mm_Vertical
Changed lines of the file:
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@@
       (effects (font (size 1.27 1.27)) (justify right))
     )
-    (property "Footprint" "" (at 175.26 66.675 0)
+    (property "Footprint" "Connector_PinHeader_2.54mm:PinHeader_1x04_P2.54mm_Vertical" (at 175.26 66.675 0)
       (effects (font (size 1.27 1.27)) hide)
     )
@@
       (effects (font (size 1.27 1.27)) hide)
     )
-    (pin "2")
-    (pin "4")
-    (pin "3")
-    (pin "1")
+    (pin "1")
+    (pin "2")
+    (pin "3")
+    (pin "4")
     (instances
       (project "EPROM 2716 Program Voltage Booster"
@@
       (effects (font (size 1.27 1.27)) hide)
     )
-    (pin "2")
-    (pin "5")
-    (pin "4")
-    (pin "1")
-    (pin "6")
-    (pin "3")
+    (pin "1")
+    (pin "2")
+    (pin "3")
+    (pin "4")
+    (pin "5")
+    (pin "6")
     (instances
       (project "EPROM 2716 Program Voltage Booster"
@@
       (effects (font (size 1.27 1.27)) hide)
     )
-    (pin "20")
-    (pin "18")
-    (pin "12")
-    (pin "17")
-    (pin "9")
-    (pin "8")
-    (pin "3")
-    (pin "15")
-    (pin "22")
-    (pin "7")
-    (pin "23")
-    (pin "14")
-    (pin "5")
-    (pin "21")
-    (pin "4")
-    (pin "16")
-    (pin "11")
-    (pin "10")
-    (pin "2")
-    (pin "6")
-    (pin "1")
-    (pin "19")
-    (pin "24")
-    (pin "13")
-    (instances
-      (project "EPROM 2716 Program Voltage Booster"
-        (path "/c4e9ad1c-aedb-4321-a3b6-fc92e425bf09"
-          (reference "U1") (unit 1)
-        )
-      )
-    )
-  )
-  (symbol (lib_id "ForgottenMachines:2716_EPROM") (at 232.41 63.5 0) (unit 1)
-    (in_bom yes) (on_board yes) (dnp no)
-    (property "Reference" "P1" (at 230.505 66.04 0)
-      (effects (font (size 1.27 1.27)) (justify left))
-    )
-    (property "Value" "2716_EPROM" (at 226.06 74.295 0)
-      (effects (font (size 1.27 1.27)) (justify left))
-    )
-    (property "Footprint" "Package_DIP:DIP-24_W15.24mm" (at 265.43 113.03 0)
-      (effects (font (size 1.27 1.27)) hide)
-    )
-    (property "Datasheet" "" (at 280.67 109.22 0)
-      (effects (font (size 1.27 1.27)) hide)
-    )
-    (pin "13")
-    (pin "9")
-    (pin "7")
+    (pin "1")
     (pin "10")
     (pin "11")
+    (pin "12")
+    (pin "13")
     (pin "14")
-    (pin "24")
-    (pin "3")
-    (pin "5")
+    (pin "15")
+    (pin "16")
     (pin "17")
+    (pin "18")
+    (pin "19")
+    (pin "2")
     (pin "20")
     (pin "21")
-    (pin "4")
-    (pin "6")
+    (pin "22")
+    (pin "23")
+    (pin "24")
+    (pin "3")
+    (pin "4")
+    (pin "5")
+    (pin "6")
+    (pin "7")
     (pin "8")
-    (pin "18")
-    (pin "23")
-    (pin "2")
-    (pin "22")
+    (pin "9")
+    (instances
+      (project "EPROM 2716 Program Voltage Booster"
+        (path "/c4e9ad1c-aedb-4321-a3b6-fc92e425bf09"
+          (reference "U1") (unit 1)
+        )
+      )
+    )
+  )
+  (symbol (lib_id "ForgottenMachines:2716_EPROM") (at 232.41 63.5 0) (unit 1)
+    (in_bom yes) (on_board yes) (dnp no)
+    (property "Reference" "P1" (at 230.505 66.04 0)
+      (effects (font (size 1.27 1.27)) (justify left))
+    )
+    (property "Value" "2716_EPROM" (at 226.06 74.295 0)
+      (effects (font (size 1.27 1.27)) (justify left))
+    )
+    (property "Footprint" "Package_DIP:DIP-24_W15.24mm" (at 265.43 113.03 0)
+      (effects (font (size 1.27 1.27)) hide)
+    )
+    (property "Datasheet" "" (at 280.67 109.22 0)
+      (effects (font (size 1.27 1.27)) hide)
+    )
+    (pin "1")
+    (pin "10")
+    (pin "11")
     (pin "12")
+    (pin "13")
+    (pin "14")
     (pin "15")
     (pin "16")
+    (pin "17")
+    (pin "18")
     (pin "19")
-    (pin "1")
+    (pin "2")
+    (pin "20")
+    (pin "21")
+    (pin "22")
+    (pin "23")
+    (pin "24")
+    (pin "3")
+    (pin "4")
+    (pin "5")
+    (pin "6")
+    (pin "7")
+    (pin "8")
+    (pin "9")
     (instances
       (project "EPROM 2716 Program Voltage Booster"
@@
       (effects (font (size 1.27 1.27)) hide)
     )
-    (pin "2")
-    (pin "5")
-    (pin "4")
-    (pin "1")
-    (pin "6")
-    (pin "3")
+    (pin "1")
+    (pin "2")
+    (pin "3")
+    (pin "4")
+    (pin "5")
+    (pin "6")
     (instances
       (project "EPROM 2716 Program Voltage Booster"
@@
       (effects (font (size 1.27 1.27)) hide)
     )
-    (pin "2")
-    (pin "1")
+    (pin "1")
+    (pin "2")
     (pin "3")
     (instances
@@
       (effects (font (size 1.27 1.27)) hide)
     )
-    (pin "2")
-    (pin "1")
-    (instances
-      (project "EPROM 2716 Program Voltage Booster"
+    (pin "1")
+    (pin "2")
+    (instances
+      (project "EPROM 2716 Program Voltage Booster"

Commit message: 2716 Adapter
Parts:
- BT1: footprint (none) -> Forgotten Machines:9v Battery PCB-Mount
- SW1: footprint (none) -> Forgotten Machines:SW_Slide_DPDT
Other:
- note added: "Inadequate TL866A +15v Programmer Voltage"
- moved on the sheet: MES1
Changed lines of the file:
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@@
     (stroke (width 0) (type default))
+  )
+  (rectangle (start 152.4 28.575) (end 152.4 62.865)
+    (stroke (width 0) (type default))
+    (fill (type none))
+  )
+  (text "Inadequate TL866A +15v\nProgrammer Voltage" (at 159.385 29.21 0)
+    (effects (font (size 1.27 1.27)) (justify left bottom))
   )
   (label "Vpp from TL866A" (at 211.455 29.845 0) (fields_autoplaced)
@@
     )
   )
-  (global_label "GND" (shape input) (at 54.61 35.56 270) (fields_autoplaced)
-    (effects (font (size 1.27 1.27)) (justify right))
-    (property "Intersheetrefs" "${INTERSHEET_REFS}" (at 54.61 41.7615 90)
+  (global_label "GND" (shape input) (at 40.64 33.02 270) (fields_autoplaced)
+    (effects (font (size 1.27 1.27)) (justify right))
+    (property "Intersheetrefs" "${INTERSHEET_REFS}" (at 40.64 39.2215 90)
       (effects (font (size 1.27 1.27)) (justify right) hide)
     )
@@
     )
   )
-  (global_label "+24V" (shape input) (at 54.61 22.86 90) (fields_autoplaced)
-    (effects (font (size 1.27 1.27)) (justify left))
-    (property "Intersheetrefs" "${INTERSHEET_REFS}" (at 54.61 15.449 90)
-      (effects (font (size 1.27 1.27)) (justify left) hide)
-    )
-  )
-  (global_label "+5V" (shape input) (at 63.5 29.21 0) (fields_autoplaced)
-    (effects (font (size 1.27 1.27)) (justify left))
-    (property "Intersheetrefs" "${INTERSHEET_REFS}" (at 69.7015 29.21 0)
+  (global_label "+24V" (shape input) (at 40.64 20.32 90) (fields_autoplaced)
+    (effects (font (size 1.27 1.27)) (justify left))
+    (property "Intersheetrefs" "${INTERSHEET_REFS}" (at 40.64 12.909 90)
+      (effects (font (size 1.27 1.27)) (justify left) hide)
+    )
+  )
+  (global_label "+5V" (shape input) (at 49.53 26.67 0) (fields_autoplaced)
+    (effects (font (size 1.27 1.27)) (justify left))
+    (property "Intersheetrefs" "${INTERSHEET_REFS}" (at 55.7315 26.67 0)
       (effects (font (size 1.27 1.27)) (justify left) hide)
     )
@@
   )
   (symbol (lib_id "Connector:Conn_01x04_Pin") (at 175.26 66.675 180) (unit 1)
-    (in_bom yes) (on_board yes) (dnp no) (fields_autoplaced)
-    (property "Reference" "J1" (at 177.165 64.135 0)
+    (in_bom yes) (on_board yes) (dnp no)
+    (property "Reference" "J1" (at 170.815 71.12 0)
       (effects (font (size 1.27 1.27)) (justify right))
     )
-    (property "Value" "External Power for Vpp" (at 177.165 66.675 0)
+    (property "Value" "External Power for Vpp" (at 176.53 75.565 90)
       (effects (font (size 1.27 1.27)) (justify right))
     )
@@
       (effects (font (size 1.27 1.27)))
     )
-    (property "Footprint" "" (at 152.4 64.135 0)
+    (property "Footprint" "Forgotten Machines:SW_Slide_DPDT" (at 152.4 64.135 0)
       (effects (font (size 1.27 1.27)) hide)
     )
@@
       (effects (font (size 1.27 1.27)))
     )
-    (property "Footprint" "" (at 152.4 29.845 0)
+    (property "Footprint" "Forgotten Machines:SW_Slide_DPDT" (at 152.4 29.845 0)
       (effects (font (size 1.27 1.27)) hide)
     )
@@
     )
   )
-  (symbol (lib_id "ForgottenMachines:Voltmeter Cheap Amazon") (at 50.165 29.21 0) (unit 1)
+  (symbol (lib_id "ForgottenMachines:Voltmeter Cheap Amazon") (at 36.195 26.67 0) (unit 1)
     (in_bom yes) (on_board yes) (dnp no) (fields_autoplaced)
-    (property "Reference" "MES1" (at 49.53 28.048 0)
+    (property "Reference" "MES1" (at 35.56 25.508 0)
       (effects (font (size 1.27 1.27)) (justify right))
     )
-    (property "Value" "Cheap Amazon Voltmeter" (at 49.53 30.588 0)
+    (property "Value" "Cheap Amazon Voltmeter" (at 35.56 28.048 0)
       (effects (font (size 1.27 1.27)) (justify right))
     )
-    (property "Footprint" "Forgotten Machines:Cheap Amazon Voltmeter" (at 16.51 21.59 0)
-      (effects (font (size 1.27 1.27)) hide)
-    )
-    (property "Datasheet" "~" (at 31.75 27.94 90)
+    (property "Footprint" "Forgotten Machines:Cheap Amazon Voltmeter" (at 2.54 19.05 0)
+      (effects (font (size 1.27 1.27)) hide)
+    )
+    (property "Datasheet" "~" (at 17.78 25.4 90)
       (effects (font (size 1.27 1.27)) hide)
     )
@@
       (effects (font (size 1.27 1.27)))
     )
-    (property "Footprint" "" (at 119.761 33.02 90)
-      (effects (font (size 1.27 1.27)) hide)
-    )
+    (property "Footprint" "Forgotten Machines:9v Battery PCB-Mount" (at 119.761 33.02 90)
+      (effects (font (size 1.27 1.27)) hide)
+    )

Commit message: lots-o-stuff
Parts:
- added C1: 100nF, Forgotten Machines:Disc Capacitor Common Entrex Trapezoid, symbol ForgottenMachines:CAP_Disc_Common_-_Entrex_Trapezoid
- added C2: 47μF 35V, Capacitor_THT:CP_Radial_D5.0mm_P2.50mm, symbol Device:C_Polarized
Connections:
- net +24V: now also MES1.3, C1.1, C2.1; no longer MES1.1
- net +5V: now also MES1.2 (PWR); no longer MES1.3 (PWR)
- net GND: now also MES1.1, C1.2, C2.2; no longer MES1.2
Other:
- note added: "To Reader/Programmer Socket"
