File: DIP Socket Adaptor - EEPROM/2716 to 82S129.kicad_pcb (KiCad board)
At the start: 2 copper layers, 45.7 x 45.7 mm, 7 parts, among them J1 Conn_02x14_Counter_Clockwise, J2 Conn_01x14, J3 Conn_01x14, J4 Conn_01x14, J5 Conn_01x14, J6 Conn_01x14, J7 Conn_01x14

Commit message: 82S129/6
Parts:
- removed J1: Conn_02x14_Counter_Clockwise, Package_DIP:DIP-28_W15.24mm_Socket
- removed J2, J3, J6, J7: Conn_01x14, Connector Board:PinHeader_1x14_P2.54mm_Vertical
- removed J4, J5: Conn_01x14, Connector Board:PinHeader_1x14_P2.54mm_Vertical2
- added U1: 2716_EPROM, Package_DIP:DIP-24_W15.24mm, F.Cu at (141.6, 59.7)
- added U2: 82S126, Package_DIP:DIP-16_W7.62mm, F.Cu at (145.4, 61.6)
Routing:
- net GND: track 0.00 -> 33.7 mm
- net O3: track 0.00 -> 15.6 mm
- net 9: track 15.2 -> 0.00 mm
- net 8: track 15.2 -> 0.00 mm
- net 7: track 15.2 -> 0.00 mm
- net 6: track 15.2 -> 0.00 mm
- net 5: track 15.2 -> 0.00 mm
- net 4: track 15.2 -> 0.00 mm
- net 3: track 15.2 -> 0.00 mm
- net 28: track 15.2 -> 0.00 mm
- net 27: track 15.2 -> 0.00 mm
- net 26: track 15.2 -> 0.00 mm
- net 25: track 15.2 -> 0.00 mm
- net 24: track 15.2 -> 0.00 mm
- net 23: track 15.2 -> 0.00 mm
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- added copper zone on B.Cu, net GND
Other:
- board text added: "2716 to 82S126/129 Adapter"
- board text removed: "EPROM Pinout Universal Adapter"
- board text removed: "FORGOTTEN MACHINES"

Commit message: atx
Changed lines of the file:
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@@
       (xy 136.955684 66.741825)
       (xy 136.955684 66.741826)
-      (xy 136.955684 66.741826)
       (xy 136.955683 66.741827)
       (xy 136.955682 66.741827)
@@
       (xy 132.218145 59.203811)
       (xy 132.218145 59.203813)
-      (xy 132.218145 59.203813)
       (xy 132.218144 59.203814)
       (xy 132.217053 59.208847)
@@
       (xy 136.984478 60.859657)
       (xy 136.984481 60.859656)
-      (xy 136.984481 60.859656)
       (xy 136.98448 60.859658)
       (xy 136.984479 60.859659)
@@
   )
   (dimension (type aligned) (layer "Dwgs.User")
-    (pts (xy 171.45 95.25) (xy 171.45 49.53))
+    (pts (xy 172.72 95.25) (xy 172.72 49.53))
     (height 1.27)
-    (gr_text "45.7200 mm" (at 171.57 72.39 90) (layer "Dwgs.User")
+    (gr_text "45.7200 mm" (at 172.84 72.39 90) (layer "Dwgs.User")
       (effects (font (size 1 1) (thickness 0.15)))
     )
