File: DIP Socket Adaptor - EEPROM/EPROM 2716 Program Voltage Booster.kicad_pcb (KiCad board)
At the start: 2 copper layers, 45.7 x 45.7 mm, 7 parts, among them J1 Conn_02x14_Counter_Clockwise, J2 Conn_01x14, J3 Conn_01x14, J4 Conn_01x14, J5 Conn_01x14, J6 Conn_01x14, J7 Conn_01x14

Commit message: 2716 Adapter
Parts:
- removed J2, J3, J6, J7: Conn_01x14, Connector Board:PinHeader_1x14_P2.54mm_Vertical
- removed J4, J5: Conn_01x14, Connector Board:PinHeader_1x14_P2.54mm_Vertical2
- added BT1: 9v Battery, Forgotten Machines:9v Battery PCB-Mount, F.Cu at (211.5, 81.3)
- added D1: 1N4004, Diode_THT:D_DO-41_SOD81_P10.16mm_Horizontal, F.Cu at (202.6, 103.5)
- added D2: 1N4004, Diode_THT:D_DO-41_SOD81_P10.16mm_Horizontal, F.Cu at (203.2, 82.5)
- added MES1: Cheap Amazon Voltmeter, Forgotten Machines:Cheap Amazon Voltmeter, F.Cu at (196.2, 113.5)
- added P1: 2716_EPROM, Package_DIP:DIP-24_W15.24mm, F.Cu at (184.8, 74.3)
- added SW1: Voltage Boost, Forgotten Machines:SW_Slide_DPDT, F.Cu at (215.3, 115.5)
- added U1: 2716_EPROM, Package_DIP:DIP-24_W15.24mm, F.Cu at (179.7, 74.3)
- J1: value Conn_02x14_Counter_Clockwise -> External Power for Vpp; footprint Package_DIP:DIP-28_W15.24mm_Socket -> Connector_PinHeader_2.54mm:PinHeader_1x04_P2.54mm_Vertical
- moved J1 68.1 mm to (208.9, 69.8), turned to 90 degrees
Connections:
- J1 pad 1: 1 -> GND
- J1 pad 2: 2 -> GND
- J1 pad 3: 3 -> Net-(J1-Pin_3)
- J1 pad 4: 4 -> Net-(J1-Pin_3)
Routing:
- net +24V: track 0.00 -> 67.4 mm
- net +5V: track 0.00 -> 54.4 mm
- net Net-(J1-Pin_3): track 0.00 -> 40.0 mm
- net Vpp from TL866A: track 0.00 -> 37.4 mm
- net Net-(BT1-+): track 0.00 -> 26.7 mm
- net Net-(D2-A): track 0.00 -> 22.8 mm
- net 9: track 15.2 -> 0.00 mm
- net 8: track 15.2 -> 0.00 mm
- net 7: track 15.2 -> 0.00 mm
- net 6: track 15.2 -> 0.00 mm
- net 5: track 15.2 -> 0.00 mm
- net 4: track 15.2 -> 0.00 mm
- net 3: track 15.2 -> 0.00 mm
- net 28: track 15.2 -> 0.00 mm
- net 27: track 15.2 -> 0.00 mm
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- added copper zone on B.Cu, net GND
- added copper zone on F.Cu, net GND
Other:
- board size 45.7 x 45.7 mm -> 46.4 x 59.1 mm
- board text added: "+"
- board text added: "9-Volt Battery"
- board text added: "External Vpp Source"
- board text added: "GND"
- board text removed: "EPROM Pinout Universal Adapter"
- board text removed: "FORGOTTEN MACHINES"

Commit message: build
Parts:
- moved MES1 2.51 mm to (193.7, 113.7)
Routing:
- net Net-(J1-Pin_3): track 40.0 -> 48.9 mm
- net +5V: track 54.4 -> 55.5 mm
- net +24V: track 67.4 -> 68.6 mm
Other:
- board text added: "2716 EPROM Programming Voltage Booster"
- board text added: "ADD a {dblquote}Mega{dblquote} version with 3 or 4 9v batteries and an adjustable voltage regulator"
- board text added: "For use with MiniPro TL866A and similar programmers"
- board text added: "Program Boost"
- board text added: "Read/ Normal"
Changed lines of the file:
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@@
     (property "Sheetname" "")
     (attr through_hole)
-    (fp_text reference "P1" (at 7.62 -2.33) (layer "F.SilkS")
+    (fp_text reference "P1" (at 6.985 0.635) (layer "F.SilkS") hide
         (effects (font (size 1 1) (thickness 0.15)))
     )
@@
         (effects (font (size 1 1) (thickness 0.15)))
     )
-    (fp_text value "Voltage Boost" (at -14.5 2 90) (layer "F.Fab")
-        (effects (font (size 1 1) (thickness 0.15)))
-    )
-    (fp_text user "${REFERENCE}" (at -14.5 -1.5 90) (layer "F.Fab")
+    (fp_text value "Voltage Boost" (at 2.46 14.5525 90) (layer "F.Fab")
+        (effects (font (size 1 1) (thickness 0.15)))
+    )
+    (fp_text user "${REFERENCE}" (at 3.095 12.0125 90) (layer "F.Fab")
         (effects (font (size 1 1) (thickness 0.15)))
     )
@@
   )
   (footprint "Forgotten Machines:Cheap Amazon Voltmeter" (layer "F.Cu")
-    (at 196.215 113.535)
+    (at 193.705 113.665)
     (property "Sheetfile" "EPROM 2716 Program Voltage Booster.kicad_sch")
     (property "Sheetname" "")
@@
     (property "Sheetname" "")
     (attr through_hole)
-    (fp_text reference "U1" (at 7.62 -2.33) (layer "F.SilkS")
+    (fp_text reference "U1" (at 8.26 0.64) (layer "F.SilkS") hide
         (effects (font (size 1 1) (thickness 0.15)))
     )
@@
   (gr_rect (start 175.895 66.04) (end 222.25 125.095)
     (stroke (width 0.05) (type default)) (fill none) (layer "Edge.Cuts"))
-  (gr_text "ForgottenMachines.com" (at 207.01 142.875) (layer "F.SilkS")
-    (effects (font (size 1.5 1.5) (thickness 0.2)))
+  (gr_text "ForgottenMachines.com" (at 210.185 123.19) (layer "F.SilkS")
+    (effects (font (size 1.3 1.3) (thickness 0.2)))
+  )
+  (gr_text "Read/\nNormal" (at 220.66 117.86 90) (layer "F.SilkS")
+    (effects (font (size 0.75 0.75) (thickness 0.17) bold))
   )
   (gr_text "9-Volt Battery" (at 220.345 92.075 90) (layer "F.SilkS")
@@
     (effects (font (size 1 1) (thickness 0.2) bold) (justify left bottom))
   )
+  (gr_text "2716 EPROM \nProgramming Voltage\nBooster" (at 190.5 69.85) (layer "F.SilkS")
+    (effects (font (size 1.3 1.3) (thickness 0.2)))
+  )
+  (gr_text "Program\nBoost" (at 220.66 108.335 90) (layer "F.SilkS")
+    (effects (font (size 0.75 0.75) (thickness 0.17) bold))
+  )
   (gr_text "+" (at 215.9 72.39) (layer "F.SilkS")
     (effects (font (size 1 1) (thickness 0.2) bold) (justify left bottom))
   )
+  (gr_text "For use with \nMiniPro TL866A\nand similar programmers" (at 189.865 88.265 90) (layer "F.SilkS")
+    (effects (font (size 1.3 1.3) (thickness 0.2)))
+  )
   (gr_text "External Vpp Source" (at 205.74 67.945) (layer "F.SilkS")
     (effects (font (size 1 1) (thickness 0.15)) (justify left bottom))
+  )
+  (gr_text "ADD a {dblquote}Mega{dblquote} version with 3 or 4 9v batteries\n and an adjustable voltage regulator" (at 196.85 133.35) (layer "Dwgs.User")
+    (effects (font (size 1 1) (thickness 0.15)) (justify bottom))
   )
   (dimension (type aligned) (layer "Edge.Cuts")
@@
     (style (thickness 0.05) (arrow_length 1.27) (text_position_mode 0) (extension_height 0.58642) (extension_offset 0.5) keep_text_aligned)
   )
+  (segment (start 196.245 119.35) (end 196.245 123.165) (width 0.25) (layer "B.Cu") (net 1))
   (segment (start 197.485 84.455) (end 197.485 101.462767) (width 0.5) (layer "B.Cu") (net 1))
   (segment (start 197.485 101.462767) (end 199.527233 103.505) (width 0.5) (layer "B.Cu") (net 1))
   (segment (start 198.755 104.277233) (end 199.527233 103.505) (width 0.25) (layer "B.Cu") (net 1))
+  (segment (start 198.755 116.84) (end 198.755 104.277233) (width 0.25) (layer "B.Cu") (net 1))
   (segment (start 200.66 103.505) (end 202.565 103.505) (width 0.5) (layer "B.Cu") (net 1))
   (segment (start 213.36 113.5325) (end 215.3175 115.49) (width 0.5) (layer "B.Cu") (net 1))
   (segment (start 205.74 103.505) (end 213.36 111.125) (width 0.5) (layer "B.Cu") (net 1))
+  (segment (start 198.755 116.84) (end 196.245 119.35) (width 0.25) (layer "B.Cu") (net 1))
   (segment (start 200.66 103.505) (end 205.74 103.505) (width 0.5) (layer "B.Cu") (net 1))
   (segment (start 199.527233 103.505) (end 200.66 103.505) (width 0.5) (layer "B.Cu") (net 1))
-  (segment (start 198.755 123.035) (end 198.755 104.277233) (width 0.25) (layer "B.Cu") (net 1))
   (segment (start 194.94 81.91) (end 197.485 84.455) (width 0.5) (layer "B.Cu") (net 1))
   (segment (start 213.36 111.125) (end 213.36 113.5325) (width 0.5) (layer "B.Cu") (net 1))
@@
   (segment (start 203.2 98.3725) (end 215.3175 110.49) (width 0.5) (layer "F.Cu") (net 4))
   (segment (start 203.2 92.71) (end 203.2 98.3725) (width 0.5) (layer "F.Cu") (net 4))
-  (segment (start 219.6825 111.125) (end 221.035 109.7725) (width 0.75) (layer "B.Cu") (net 6))
   (segment (start 221.035 109.7725) (end 221.035 74.35) (width 0.75) (layer "B.Cu") (net 6))
-  (segment (start 219.6825 111.125) (end 217.8175 112.99) (width 0.75) (layer "B.Cu") (net 6))
+  (segment (start 219.075 72.39) (end 216.535 69.85) (width 0.75) (layer "B.Cu") (net 6))
+  (segment (start 216.535 69.85) (end 213.995 69.85) (width 0.75) (layer "B.Cu") (net 6))
+  (segment (start 217.8175 112.99) (end 221.035 109.7725) (width 0.75) (layer "B.Cu") (net 6))
+  (segment (start 221.035 74.35) (end 219.075 72.39) (width 0.75) (layer "B.Cu") (net 6))
   (segment (start 200.02 74.29) (end 200.025 74.295) (width 0.25) (layer "F.Cu") (net 7))
   (segment (start 194.94 74.29) (end 200.02 74.29) (width 1.5) (layer "F.Cu") (net 7))
-  (segment (start 193.675 123.035) (end 193.675 75.555) (width 0.5) (layer "B.Cu") (net 7))
+  (segment (start 193.675 120.655) (end 191.165 123.165) (width 0.5) (layer "B.Cu") (net 7))
+  (segment (start 193.675 117.475) (end 193.675 75.555) (width 0.5) (layer "B.Cu") (net 7))
+  (segment (start 193.675 117.475) (end 193.675 120.655) (width 0.5) (layer "B.Cu") (net 7))
   (segment (start 193.675 75.555) (end 194.94 74.29) (width 0.5) (layer "B.Cu") (net 7))
   (segment (start 179.7 74.29) (end 184.78 74.29) (width 0.25) (layer "F.Cu") (net 8))
@@
     (polygon
       (pts
-        (xy 175.895 69.215)
+        (xy 175.895 66.04)
         (xy 175.895 125.73)
         (xy 222.25 125.73)
-        (xy 222.25 69.215)
+        (xy 222.25 66.04)
       )
     )
@@
     (polygon
       (pts
-        (xy 175.895 69.215)
+        (xy 175.895 66.04)
         (xy 175.895 125.73)
         (xy 222.25 125.73)
-        (xy 222.25 69.215)
+        (xy 222.25 66.04)
       )
     )

Commit message: lots-o-stuff
Parts:
- added C1: 100nF, Forgotten Machines:Disc Capacitor Common Entrex Trapezoid, F.Cu at (200.4, 85.1)
- added C2: 47μF 35V, Capacitor_THT:CP_Radial_D5.0mm_P2.50mm, F.Cu at (200.1, 77.5)
- moved MES1 8.67 mm to (191.1, 121.9)
- moved D1 8.64 mm to (200.0, 111.8)
- moved D2 8.64 mm to (200.7, 90.8)
- moved SW1 8.64 mm to (212.8, 123.7)
- moved P1 8.64 mm to (182.2, 82.5)
- moved U1 8.64 mm to (177.2, 82.5)
- moved J1 8.47 mm to (207.0, 78.1)
- moved BT1 8.34 mm to (210.2, 89.5)
Connections:
- MES1 pad 1: +24V -> GND
- MES1 pad 2: GND -> +5V
- MES1 pad 3: +5V -> +24V
Routing:
- net +24V: track 68.6 -> 96.6 mm
- net Net-(BT1-+): track 26.7 -> 31.7 mm
- net Net-(BT1--): track 8.78 -> 13.2 mm
- net +5V: track 55.5 -> 54.5 mm
