File: MFM_ST506 Breakout Board/MFM_ST506 Breakout Board.kicad_pcb (KiCad board)
At the start: 2 copper layers, 195.6 x 87.6 mm, 45 parts, among them J1 Conn_02x10_Odd_Even, J10 Conn_02x17_Odd_Even, J11 Conn_01x09, J12 Conn_01x09, J13 Conn_01x09, J14 Conn_01x09, J15 Conn_01x10, J16 Conn_01x10, J17 Conn_01x10, J18 Conn_01x10, J19 Conn_01x07, J2 Conn_02x10_Odd_Even, J20 Conn_01x07, J21 Conn_01x06, J22 Conn_01x07, J23 Conn_02x25_Odd_Even, J24 Conn_02x25_Odd_Even, J25 Conn_01x08, J26 Conn_01x08, J27 Conn_01x08, J28 Conn_01x08, J3 Conn_02x10_Odd_Even, J4 Conn_02x10_Odd_Even, J41 Conn_01x07, J42 Conn_01x06, J43 Conn_01x05, J44 Conn_01x04, J45 Conn_01x03, J46 Conn_01x05, J47 Conn_01x04, J48 Conn_01x03, J49 Conn_01x06, J5 Conn_02x25_Odd_Even, J50 Conn_01x05, J51 Conn_01x04, J52 Conn_01x03, J53 Conn_01x06, J54 Conn_01x05, J55 Conn_01x04, J56 Conn_01x03, J6 Conn_02x25_Odd_Even, J7 Conn_02x17_Odd_Even, J8 Conn_02x17_Odd_Even, J9 Conn_02x17_Odd_Even

Commit message: atx
Parts:
- removed G***: LOGO, MFM_ST506 Breakout Board:forgotten machines text
Other:
- board text added: "20, 34 & 50-pin Breakout Board"
